File: kicad/cymometer.kicad_pcb (KiCad board)
At the start: 2 copper layers, 88.4 x 62 mm, 60 parts, among them IC1 ATMEGA8-P, P1 BNC, P2 CONN_2, P3 CONN_3X2, Q1 BC550, SW1 SW_PUSH, SW2 SPST, SW3 SW_PUSH, U1 7805, X1 20.48 MГц

Commit message: Add all
Parts:
- moved AFF1 137.1 mm to (152.0, 33.1)
- moved SW2 136.4 mm to (69.0, 26.9), turned to 90 degrees
- moved AFF2 126.0 mm to (144.4, 33.1)
- moved C10 121.3 mm to (99.1, 65.0), turned to 180 degrees
- moved AFF3 113.9 mm to (136.8, 33.1)
- moved AFF8 112.9 mm to (98.7, 33.1)
- moved SW1 109.6 mm to (69.6, 41.8), turned to 90 degrees
- moved D4 108.8 mm to (92.8, 37.0)
- moved D3 108.4 mm to (92.8, 29.3)
- moved AFF4 107.2 mm to (129.2, 33.1)
- moved AFF7 106.1 mm to (106.3, 33.1)
- moved AFF5 103.6 mm to (121.5, 33.1)
- moved AFF6 102.9 mm to (113.9, 33.1)
- moved SW3 84.0 mm to (69.5, 58.3), turned to 90 degrees
- moved R12 73.4 mm to (87.9, 26.4), turned to 180 degrees
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Connections:
- AFF2 pad 3: (no net) -> Net-(AFF2-Pad3)
- AFF2 pad 8: Net-(AFF2-Pad8) -> (no net)
- DD5 pad 1: Net-(D3-Pad2) -> Net-(AFF1-Pad3)
- DD5 pad 10: Net-(AFF1-Pad3) -> Net-(D3-Pad2)
- DD5 pad 2: Net-(AFF8-Pad3) -> Net-(AFF2-Pad3)
- DD5 pad 3: Net-(AFF7-Pad3) -> Net-(AFF3-Pad3)
- DD5 pad 4: Net-(AFF6-Pad3) -> Net-(AFF4-Pad3)
- DD5 pad 6: Net-(AFF4-Pad3) -> Net-(AFF6-Pad3)
- DD5 pad 7: Net-(AFF3-Pad3) -> Net-(AFF7-Pad3)
- DD5 pad 9: Net-(AFF2-Pad8) -> Net-(AFF8-Pad3)
- R3 pad 1: (no net) -> Net-(C2-Pad1)
Routing:
- net GND: track 0.00 -> 435.7 mm, vias 0 -> 2
- net VCC: track 0.00 -> 396.1 mm, vias 0 -> 3
- net Net-(AFF1-Pad7): track 0.00 -> 100.8 mm
- net Net-(DD5-Pad15): track 0.00 -> 99.4 mm
- net Net-(DD4-Pad5): track 0.00 -> 98.8 mm, vias 0 -> 3
- net Net-(DD1-Pad8): track 0.00 -> 96.6 mm
- net Net-(AFF1-Pad10): track 0.00 -> 94.6 mm
- net Net-(DD3-Pad10): track 0.00 -> 93.9 mm
- net Net-(AFF1-Pad4): track 0.00 -> 87.4 mm
- net Net-(IC1-Pad17): track 0.00 -> 87.0 mm
- net Net-(DD1-Pad13): track 0.00 -> 87.0 mm
- net Net-(AFF1-Pad6): track 0.00 -> 85.5 mm
- net Net-(AFF1-Pad1): track 0.00 -> 83.2 mm
- net Net-(DD1-Pad5): track 0.00 -> 81.0 mm
- net Net-(DD5-Pad14): track 0.00 -> 79.6 mm
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Other:
- board size 88.4 x 62 mm -> 128.4 x 62 mm

Commit message: Add all
Parts:
- moved C11 0.38 mm to (55.1, 28.6)
Routing:
- net GND: track 435.7 -> 457.6 mm
- net Net-(DD3-Pad3): track 36.2 -> 34.5 mm
Other:
- outline, holes or cut-outs redrawn
Changed lines of the file:
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@@
     (links 201)
     (no_connects 4)
-    (area 24.871 18.033 176.127571 84.179)
+    (area 28.372999 19.990999 156.920001 82.117001)
     (thickness 1.6)
-    (drawings 12)
-    (tracks 843)
+    (drawings 14)
+    (tracks 854)
     (zones 0)
     (modules 60)
@@
   )
   (module cymometer:C_Rect_L7_W2.5_P5 (layer F.Cu)
-    (at 54.737 28.575 270)
+    (at 55.118 28.575 270)
     (descr "Film Capacitor Length 7mm x Width 2.5mm, Pitch 5mm")
     (tags Capacitor)
@@
     )
   )
+  (gr_circle (center 60.5155 49.5935) (end 61.468 50.6095) (layer Edge.Cuts) (width 0.15))
+  (gr_circle (center 60.5155 49.5935) (end 61.468 50.6095) (layer Edge.Cuts) (width 0.15))
   (gr_circle (center 30.6705 22.225) (end 31.623 23.241) (layer Edge.Cuts) (width 0.15))
   (gr_circle (center 30.6705 22.225) (end 31.623 23.241) (layer Edge.Cuts) (width 0.15))
@@
   (segment (start 31.115 65.024) (end 31.496 65.405) (width 0.8) (layer B.Cu) (net 1))
   (segment (start 36.115 61.976) (end 38.608 61.976) (width 0.8) (layer B.Cu) (net 2))
+  (segment (start 38.608 24.765) (end 41.148 24.765) (width 0.8) (layer F.Cu) (net 3))
+  (segment (start 41.148 24.765) (end 43.688 24.765) (width 0.8) (layer F.Cu) (net 3))
+  (segment (start 51.308 32.385) (end 51.308 28.2575) (width 0.8) (layer F.Cu) (net 3))
+  (segment (start 41.148 26.3525) (end 41.148 24.765) (width 0.8) (layer F.Cu) (net 3))
+  (segment (start 41.91 27.1145) (end 41.148 26.3525) (width 0.8) (layer F.Cu) (net 3))
+  (segment (start 50.165 27.1145) (end 41.91 27.1145) (width 0.8) (layer F.Cu) (net 3))
+  (segment (start 51.308 28.2575) (end 50.165 27.1145) (width 0.8) (layer F.Cu) (net 3))
   (segment (start 124.159 56.388) (end 124.159 61.675) (width 0.8) (layer F.Cu) (net 3))
   (segment (start 133.858 71.374) (end 133.858 76.113) (width 0.8) (layer F.Cu) (net 3))
@@
   (segment (start 88.3285 50.038) (end 87.3125 49.022) (width 0.8) (layer B.Cu) (net 3))
   (segment (start 98.425 61.6585) (end 98.425 62.357) (width 0.8) (layer B.Cu) (net 3))
-  (segment (start 54.737 32.385) (end 54.737 36.449) (width 0.8) (layer B.Cu) (net 3))
+  (segment (start 55.118 32.385) (end 55.118 36.83) (width 0.8) (layer B.Cu) (net 3) (status 10))
   (segment (start 65.3415 26.924) (end 70.231 26.924) (width 0.8) (layer B.Cu) (net 3))
   (segment (start 64.897 27.3685) (end 65.3415 26.924) (width 0.8) (layer B.Cu) (net 3))
@@
   (segment (start 61.976 39.751) (end 64.897 36.83) (width 0.8) (layer B.Cu) (net 3))
   (segment (start 58.039 39.751) (end 61.976 39.751) (width 0.8) (layer B.Cu) (net 3))
-  (segment (start 54.737 36.449) (end 58.039 39.751) (width 0.8) (layer B.Cu) (net 3))
-  (segment (start 54.737 32.385) (end 54.737 43.942) (width 0.8) (layer F.Cu) (net 3))
-  (segment (start 54.737 43.942) (end 56.134 45.339) (width 0.8) (layer F.Cu) (net 3))
+  (segment (start 55.118 36.83) (end 58.039 39.751) (width 0.8) (layer B.Cu) (net 3))
+  (segment (start 55.118 32.385) (end 55.118 44.3865) (width 0.8) (layer F.Cu) (net 3) (status 10))
+  (segment (start 55.118 44.3865) (end 56.134 45.339) (width 0.8) (layer F.Cu) (net 3))
   (segment (start 154.432 75.946) (end 147.457 75.946) (width 0.8) (layer F.Cu) (net 3))
   (segment (start 147.457 75.946) (end 143.012 71.501) (width 0.8) (layer F.Cu) (net 3))
@@
   (segment (start 142.661 76.113) (end 143.764 77.216) (width 0.8) (layer B.Cu) (net 3))
   (segment (start 122.348 56.388) (end 124.159 56.388) (width 0.8) (layer B.Cu) (net 3))
-  (segment (start 54.737 32.385) (end 51.308 32.385) (width 0.8) (layer B.Cu) (net 3))
+  (segment (start 55.118 32.385) (end 51.308 32.385) (width 0.8) (layer B.Cu) (net 3) (status 10))
   (segment (start 53.63464 47.83836) (end 53.63464 49.06264) (width 0.8) (layer B.Cu) (net 3))
   (segment (start 53.63464 49.06264) (end 56.729 52.157) (width 0.8) (layer B.Cu) (net 3))
@@
   (segment (start 36.068 24.765) (end 36.068 24.003) (width 0.8) (layer F.Cu) (net 16))
   (segment (start 36.068 24.003) (end 37.7825 22.2885) (width 0.8) (layer F.Cu) (net 16))
-  (segment (start 52.2605 22.2885) (end 54.737 24.765) (width 0.8) (layer F.Cu) (net 16))
+  (segment (start 52.2605 22.2885) (end 55.118 24.765) (width 0.8) (layer F.Cu) (net 16) (status 20))
   (segment (start 37.7825 22.2885) (end 52.2605 22.2885) (width 0.8) (layer F.Cu) (net 16))
   (segment (start 36.068 36.957) (end 36.0045 36.957) (width 0.8) (layer F.Cu) (net 16))
@@
   (segment (start 58.6105 44.196) (end 51.435 37.0205) (width 0.8) (layer B.Cu) (net 16))
   (segment (start 51.435 37.0205) (end 49.022 37.0205) (width 0.8) (layer B.Cu) (net 16))
-  (segment (start 54.737 24.765) (end 58.7375 24.765) (width 0.8) (layer B.Cu) (net 16))
+  (segment (start 55.118 24.765) (end 58.7375 24.765) (width 0.8) (layer B.Cu) (net 16) (status 10))
   (segment (start 58.7375 24.765) (end 59.309 24.1935) (width 0.8) (layer B.Cu) (net 16))
   (segment (start 82.296 70.612) (end 79.629 70.612) (width 0.8) (layer F.Cu) (net 16))
@@
   (segment (start 104.648 68.453) (end 108.585 64.516) (width 0.8) (layer F.Cu) (net 32))
   (segment (start 108.585 64.516) (end 108.585 62.357) (width 0.8) (layer F.Cu) (net 32))
-  (segment (start 62.611 24.257) (end 62.611 27.1145) (width 0.8) (layer F.Cu) (net 33))
-  (segment (start 45.593 27.94) (end 41.148 32.385) (width 0.8) (layer F.Cu) (net 33))
-  (segment (start 61.7855 27.94) (end 45.593 27.94) (width 0.8) (layer F.Cu) (net 33))
-  (segment (start 62.611 27.1145) (end 61.7855 27.94) (width 0.8) (layer F.Cu) (net 33))
-  (segment (start 46.228 36.957) (end 46.228 32.385) (width 0.8) (layer B.Cu) (net 33))
-  (segment (start 46.228 32.385) (end 43.688 32.385) (width 0.8) (layer B.Cu) (net 33))
-  (segment (start 43.688 32.385) (end 41.148 32.385) (width 0.8) (layer B.Cu) (net 33))
+  (segment (start 62.611 24.257) (end 62.611 28.2575) (width 0.8) (layer F.Cu) (net 33) (status 400000))
+  (segment (start 52.6415 34.798) (end 46.228 34.798) (width 0.8) (layer F.Cu) (net 33))
+  (segment (start 53.34 34.0995) (end 52.6415 34.798) (width 0.8) (layer F.Cu) (net 33))
+  (segment (start 53.34 31.115) (end 53.34 34.0995) (width 0.8) (layer F.Cu) (net 33))
+  (segment (start 54.356 30.099) (end 53.34 31.115) (width 0.8) (layer F.Cu) (net 33))
+  (segment (start 60.7695 30.099) (end 54.356 30.099) (width 0.8) (layer F.Cu) (net 33))
+  (segment (start 62.611 28.2575) (end 60.7695 30.099) (width 0.8) (layer F.Cu) (net 33))
+  (segment (start 41.148 32.385) (end 43.688 32.385) (width 0.8) (layer F.Cu) (net 33) (status C00000))
+  (segment (start 43.688 32.385) (end 46.228 32.385) (width 0.8) (layer F.Cu) (net 33) (status C00000))
+  (segment (start 46.228 32.385) (end 46.228 34.798) (width 0.8) (layer F.Cu) (net 33) (status 400000))
+  (segment (start 46.228 34.798) (end 46.228 36.957) (width 0.8) (layer F.Cu) (net 33) (status 800000))
   (segment (start 111.125 54.737) (end 111.125 54.2925) (width 0.8) (layer F.Cu) (net 34))
   (segment (start 111.125 54.2925) (end 109.309549 52.477049) (width 0.8) (layer F.Cu) (net 34))

Commit message: Add all
Routing:
- net GND: track 457.6 -> 477.8 mm, vias 2 -> 1
- net Net-(IC1-Pad18): track 55.1 -> 67.8 mm
- net (no net): track 0.00 -> 5.08 mm
- net Net-(DD5-Pad13): track 65.7 -> 62.9 mm
- net Net-(DD2-Pad12): track 47.3 -> 44.7 mm
- net Net-(DD5-Pad12): track 60.1 -> 58.3 mm
- net Net-(DD4-Pad5): track 98.8 -> 100.3 mm
- net Net-(DD1-Pad9): track 49.4 -> 50.6 mm
- net Net-(IC1-Pad23): track 36.2 -> 37.1 mm
- net Net-(IC1-Pad24): track 22.7 -> 23.6 mm
- net Net-(DD2-Pad9): track 25.2 -> 24.5 mm, vias 1 -> 0
- net Net-(IC1-Pad19): vias 2 -> 1

Commit message: End board
Parts:
- AFF1, AFF2, AFF3, AFF4, AFF5, AFF6, AFF7, AFF8, D3, D4, DD5, SW1, SW2, SW3: moved to B.Cu
- moved D4 59.9 mm to (152.8, 36.7)
- moved D3 59.9 mm to (152.7, 29.1)
- moved C13 19.6 mm to (133.2, 53.2)
- moved DD5 15.4 mm to (135.4, 49.4)
- moved AFF1 4.64 mm to (147.4, 33.0), turned to 180 degrees
- moved AFF2 4.64 mm to (139.8, 33.0), turned to 180 degrees
- moved AFF3 4.64 mm to (132.1, 33.0), turned to 180 degrees
- moved AFF5 4.64 mm to (116.9, 33.0), turned to 180 degrees
- moved AFF7 4.64 mm to (101.7, 33.0), turned to 180 degrees
- moved AFF8 4.64 mm to (94.0, 33.0), turned to 180 degrees
- moved AFF4 4.64 mm to (124.5, 33.0), turned to 180 degrees
- moved AFF6 4.64 mm to (109.3, 33.0), turned to 180 degrees
- moved R13 0.28 mm to (87.8, 38.9)
- moved R12 0.28 mm to (87.8, 26.7)
- moved R16 0.28 mm to (87.8, 23.6)
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Connections:
- DD5 pad 1: Net-(AFF1-Pad3) -> Net-(D3-Pad2)
- DD5 pad 10: Net-(D3-Pad2) -> Net-(AFF1-Pad3)
- DD5 pad 2: Net-(AFF2-Pad3) -> Net-(AFF8-Pad3)
- DD5 pad 3: Net-(AFF3-Pad3) -> Net-(AFF7-Pad3)
- DD5 pad 4: Net-(AFF4-Pad3) -> Net-(AFF6-Pad3)
- DD5 pad 6: Net-(AFF6-Pad3) -> Net-(AFF4-Pad3)
- DD5 pad 7: Net-(AFF7-Pad3) -> Net-(AFF3-Pad3)
- DD5 pad 9: Net-(AFF8-Pad3) -> Net-(AFF2-Pad3)
Routing:
- net VCC: track 396.0 -> 347.6 mm, vias 3 -> 2
- net Net-(AFF7-Pad3): track 33.6 -> 75.1 mm
- net Net-(DD4-Pad5): track 100.3 -> 140.5 mm, vias 3 -> 1
- net Net-(D3-Pad2): track 66.3 -> 34.9 mm
- net Net-(DD5-Pad15): track 99.4 -> 69.7 mm
- net Net-(AFF2-Pad3): track 10.7 -> 39.2 mm
- net Net-(AFF1-Pad3): track 9.16 -> 28.3 mm
- net GND: track 477.8 -> 495.2 mm
- net Net-(DD5-Pad12): track 58.3 -> 72.7 mm, vias 0 -> 1
- net Net-(AFF1-Pad7): track 100.8 -> 89.8 mm
- net Net-(DD5-Pad14): track 79.6 -> 68.7 mm
- net Net-(AFF3-Pad3): track 15.3 -> 25.8 mm
- net Net-(AFF6-Pad3): track 28.4 -> 38.7 mm
- net Net-(AFF4-Pad3): track 20.4 -> 30.0 mm
- net Net-(AFF5-Pad3): track 24.8 -> 34.3 mm
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